File: board/pico-dev-v2/pico-dev.kicad_pcb (KiCad board)
At the start: 2 copper layers, 99.1 x 76.2 mm, 45 parts, among them J1 MODE, J10 SPI0, J12 SPI1/GPIO, J13 +3.3V, J14 +5V, J15 GND, J16 GND, J17 +3.3V, J18 GPIO, J19 I2S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

Commit message: pico-dev-v2 (pcb): Add missing silkscreen on analog header.
Other:
- board text added: "3.3V"
- board text added: "GP26"
- board text added: "GP27"
Changed lines of the file:
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@@
   (general
     (thickness 1.6)
-    (drawings 180)
+    (drawings 184)
     (tracks 373)
     (zones 0)
@@
       (effects (font (size 1 1) (thickness 0.15)))
     )
-    (fp_text value 10k (at 0 1.82) (layer F.SilkS)
+    (fp_text value 10k (at -0.01618 -2.14376) (layer F.SilkS)
       (effects (font (size 1 1) (thickness 0.15)))
     )
@@
     )
   )
+  (gr_text GP26 (at 154.44216 38.14064) (layer F.SilkS)
+    (effects (font (size 1 1) (thickness 0.25)))
+  )
+  (gr_text GP27 (at 154.41676 40.68064) (layer F.SilkS)
+    (effects (font (size 1 1) (thickness 0.25)))
+  )
+  (gr_text 3.3V (at 154.29992 35.96132) (layer F.SilkS)
+    (effects (font (size 1 1) (thickness 0.25)))
+  )
+  (gr_text GND (at 154.41676 43.41876) (layer F.SilkS)
+    (effects (font (size 1 1) (thickness 0.25)))
+  )
   (gr_text I2C1 (at 151.765 73.66) (layer F.SilkS)
